File: v1.0/v1.0.brd (EAGLE design)
At the start: 44.5 x 53.4 mm, 13 parts, among them IC1 1-2199298-2

Commit message: Update
Parts:
- removed JP1: (no value), pinhead:2X04
- removed JP6: (no value), pinhead:1X04
- added JP5: (no value), pinhead:2X03
- added S1: PCM12SMTR, PCM12SMTR:PCM12SMTR
- C1: value (none) -> 10uF; device adafruit:E5-6 -> rcl:E2-5
- moved C1 7.45 mm to (39.2, 31.5)
Connections:
- new net 3.3: JP3.5, S1.3
- new net 5V: JP3.4, S1.1
- net D3: no longer JP1.3, JP6.2
- net D4: no longer JP1.5, JP6.3
- net GND: now also JP5.6; no longer JP1.7, JP6.4
- net MISO: now also JP5.1; no longer JP1.6
- net MOSI: now also JP5.4; no longer JP1.8
- net RESET: now also JP5.5; no longer JP1.1
- net SCK: now also JP5.3; no longer JP1.4
- net VCC: now also JP5.2, S1.2; no longer JP1.2, JP3.4, JP6.1
Routing:
- net GND: track 98.8 -> 0.11 mm, vias 0 -> 1
- net D4: track 37.1 -> 0.00 mm, vias 1 -> 0
- net D3: track 32.1 -> 0.00 mm, vias 1 -> 0
- net 5V: track 0.00 -> 16.6 mm
- net VCC: track 63.9 -> 52.0 mm, vias 0 -> 1
- net MOSI: track 39.2 -> 30.6 mm
- net 3.3: track 0.00 -> 8.29 mm
- net MISO: track 35.2 -> 29.0 mm
- net N$1: track 11.0 -> 14.5 mm
- net RESET: track 37.3 -> 40.4 mm
- net PROG.: track 38.9 -> 39.8 mm
- added copper zone on layer 1, net GND
- added copper zone on layer 16, net GND
Other:
- board text added: "."
- board text added: "3.3V"
- board text added: "ICSP"
- board text added: "ICSP Programmer"
- board text removed: "1"
- board text removed: "8"
- board text removed: "D3"
- board text removed: "D4"
- board text removed: "GND"
